File: super7e.sch (EAGLE design)
At the start: 19 parts, among them IC1 STM32F103VCT

Commit message: *
Changed lines of the file:
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@@
 <?xml version="1.0" encoding="utf-8"?>
 <!DOCTYPE eagle SYSTEM "eagle.dtd">
-<eagle version="7.5.0">
+<eagle version="7.6.0">
 <drawing>
 <settings>
@@
 </segment>
 </net>
-<net name="N$1" class="0">
-<segment>
-<wire x1="-317.5" y1="76.2" x2="-317.5" y2="-10.16" width="0.1524" layer="91"/>
-</segment>
-</net>
-<net name="N$2" class="0">
-<segment>
-<wire x1="-281.94" y1="73.66" x2="-284.48" y2="73.66" width="0.1524" layer="91"/>
-<wire x1="-284.48" y1="73.66" x2="-284.48" y2="-10.16" width="0.1524" layer="91"/>
-</segment>
-</net>
-<net name="N$3" class="0">
-<segment>
-<wire x1="-251.46" y1="73.66" x2="-254" y2="73.66" width="0.1524" layer="91"/>
-<wire x1="-254" y1="73.66" x2="-254" y2="-12.7" width="0.1524" layer="91"/>
-</segment>
-</net>
